File: KiCad/Radio-86RK.kicad_pcb (KiCad board)
At the start: 2 copper layers, 266.7 x 203.2 mm, 188 parts, among them J1 Video, J2 5V, J3 Power, J4 Cassette, J5 Serial, J6 Parallel, Q1 2N3904, Q2 2N3904, SW1 FF, SW10 ВК CR, SW11 ЗБ DEL, SW12 LEFT, SW13 UP, SW14 RIGHT, SW15 DOWN, SW16 0, SW17 1 !, SW18 2 ", SW19 3 #, SW2 СТР CLS, SW20 4 $, SW21 5 %, SW22 6 &, SW23 7 ', SW24 8 (, SW25 9 ), SW26 : *, SW27 ; +, SW28 , <, SW29 - =, SW3 АР2 ESC, SW30 . >, SW31 / ?, SW32 Ю @, SW33 А A, SW34 Б B, SW35 Ц C, SW36 Д D, SW37 Е E, SW38 Ф F, SW39 Г G, SW4 F1, SW40 Х H, SW41 И I, SW42 Й J, SW43 К K, SW44 Л L, SW45 М M, SW46 Н N, SW47 О O, SW48 П P, SW49 Я Q, SW5 F2, SW50 Р R, SW51 С S, SW52 Т T, SW53 У U, SW54 Ж V, SW55 В W, SW56 X Ь, SW57 Ы Y, SW58 З Z, SW59 Ш [, SW6 F3, SW60 Э \, SW61 Щ ], SW62 Ч ^, SW63 SPACE, SW64 УС CTRL, SW65 CC GRAPH, SW66 RUS/LAT, SW67 Reset, SW7 F4, SW8 ТАБ TAB, SW9 ПС LF, U1 8080A/КР580ВМ80А, U10 2716/КР573РФ5, U11 2716/КР573РФ5, U12 74LS373/К555ИР22, U13 74198/К155ИР13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

Commit message: Change 8224 package to DIP16; Swap Down/Right keys; Fix U21 soviet designation
Signed-off-by: Sergey Kiselev <skiselev@gmail.com>
Parts:
- U2: footprint My_Components:IC_DIP20_300 -> My_Components:IC_DIP16_300
- U21: value TL071/К140УД6 -> TL071/КР140УД608
- moved C44 35.6 mm to (14.0, 85.1), turned to 0 degrees
- moved Y1 25.4 mm to (14.0, 80.0), turned to 180 degrees
- moved C25 21.3 mm to (14.0, 47.0), turned to 0 degrees
- moved R6 20.1 mm to (22.9, 71.1), turned to 90 degrees
- moved SW14 19.0 mm to (263.5, 200.0)
- moved SW15 19.0 mm to (244.5, 200.0)
- moved C2 16.5 mm to (14.0, 74.9)
- moved U2 12.7 mm to (14.0, 61.0)
Routing:
- net /Keyboard/K_PB7: track 439.9 -> 419.8 mm
- net /Keyboard/K_PB6: track 471.4 -> 487.1 mm
- net TTL_CLK: track 232.3 -> 217.0 mm
- net Net-(C39-Pad1): track 80.1 -> 64.8 mm
- net /READY: track 142.8 -> 127.6 mm
- net Net-(U1-Pad19): track 53.1 -> 38.1 mm
- net GND: track 2997.4 -> 2983.2 mm
- net Net-(R6-Pad2): track 17.3 -> 6.13 mm
- net RESET: track 317.3 -> 309.5 mm, vias 5 -> 4
- net VCC: track 1033.1 -> 1026.8 mm, vias 1 -> 4
- net Net-(U2-Pad15): track 20.7 -> 14.8 mm
- net OSC: track 24.4 -> 19.4 mm
- net +12V: track 270.3 -> 275.0 mm
- net Net-(U1-Pad22): track 30.7 -> 26.1 mm
- net Net-(U1-Pad15): track 37.9 -> 36.1 mm, vias 0 -> 1
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Other:
- board text added: "JLCJLCJLCJLC"
