File: KiCad/Radio-86RK-IO.kicad_sch (KiCad schematic)
At the start: 16 parts, among them J5 Serial, J6 Parallel, Q2 2N3904, U16 7486/К155ЛП5, U20 7400/К155ЛА3, U22 SN75154N/К170УП2В, U23 SN75150P/К170АП2, U24 SN75150P/К170АП2, U3 8251A/КР580ВВ51А, U4 8253/КР580ВИ53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

Commit message: Add Version 1.4 files
Signed-off-by: Sergey Kiselev <skiselev@gmail.com>
Parts:
- U6: symbol my_components:8255 -> my_components:8255A
Connections:
- net GND: now also J5.0 (GND); no longer J5.GND
Changed lines of the file:
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@@
   (title_block
     (title "Radio-86RK")
-    (date "2022-05-13")
-    (rev "1.3")
+    (date "2023-12-09")
+    (rev "1.4")
     (company "Designed by Sergey Kiselev")
     (comment 1 "Based on the previous work by Alexey Khudyakov and Radio magazine publications")
@@
     (effects (font (size 1.524 1.524)) (justify right))
   )
-  (symbol (lib_id "my_components:8255") (at 71.12 151.13 0) (unit 1)
+  (symbol (lib_id "my_components:8255A") (at 71.12 151.13 0) (unit 1)
     (in_bom yes) (on_board yes)
     (property "Reference" "U6" (id 0) (at 60.96 113.03 0))
     (property "Value" "8255A/КР580ВВ55А" (id 1) (at 58.42 115.57 0))
-    (property "Footprint" "My_Components:IC_DIP40_600" (id 2) (at 71.12 143.51 0)
-      (effects (font (size 1.27 1.27)) hide)
-    )
-    (property "Datasheet" "http://aturing.umcs.maine.edu/~meadow/courses/cos335/Intel8255A.pdf" (id 3) (at 71.12 143.51 0)
-      (effects (font (size 1.27 1.27)) hide)
+    (property "Footprint" "My_Components:IC_DIP40_600" (id 2) (at 71.12 151.13 0)
+      (effects (font (size 1.524 1.524)) hide)
+    )
+    (property "Datasheet" "http://aturing.umcs.maine.edu/~meadow/courses/cos335/Intel8255A.pdf" (id 3) (at 71.12 151.13 0)
+      (effects (font (size 1.524 1.524)) hide)
     )
     (pin "1")
@@
     )
     (property "Datasheet" "" (id 3) (at 71.12 48.26 0)
-      (effects (font (size 1.524 1.524)))
+      (effects (font (size 1.524 1.524)) hide)
     )
     (pin "1")
@@
     )
     (property "Datasheet" "" (id 3) (at 142.24 52.07 0)
-      (effects (font (size 1.524 1.524)))
+      (effects (font (size 1.524 1.524)) hide)
     )
     (pin "1")
@@
       (effects (font (size 1.524 1.524)))
     )
+    (pin "0")
     (pin "1")
     (pin "2")
@@
     (pin "8")
     (pin "9")
-    (pin "GND")
   )
   (symbol (lib_id "Device:R") (at 162.56 146.05 0) (unit 1)
