File: KiCad/Radio-86RK-Keyboard.kicad_sch (KiCad schematic)
At the start: 96 parts, among them J4 Cassette, SW1 FF, SW10 ПС LF, SW11 ВК CR, SW12 ЗБ DEL, SW13 LEFT, SW14 UP, SW15 RIGHT, SW16 DOWN, SW17 0, SW18 1 !, SW19 2 ", SW2 СТР CLS, SW20 3 #, SW21 4 $, SW22 5 %, SW23 6 &, SW24 7 ', SW25 8 (, SW26 9 ), SW27 : *, SW28 ; +, SW29 , <, SW3 АР2 ESC, SW30 - =, SW31 . >, SW32 / ?, SW33 Ю @, SW34 А A, SW35 Б B, SW36 Ц C, SW37 Д D, SW38 Е E, SW39 Ф F, SW4 F1, SW40 Г G, SW41 Х H, SW42 И I, SW43 Й J, SW44 К K, SW45 Л L, SW46 М M, SW47 Н N, SW48 О O, SW49 П P, SW5 F2, SW50 Я Q, SW51 Р R, SW52 С S, SW53 Т T, SW54 У U, SW55 Ж V, SW56 В W, SW57 X Ь, SW58 Ы Y, SW59 З Z, SW6 F3, SW60 Ш [, SW61 Э \, SW62 Щ ], SW63 Ч ^, SW64 SPACE, SW65 УС CTRL, SW66 CC GRAPH, SW67 RUS/LAT, SW7 F4, SW8 F5, SW9 ТАБ TAB, U19 7404/К155ЛН1, U21 TL071/КР140УД608, U5 8255A/КР580ВВ55А

Commit message: Updates for version v1.3: Update silkscreen and resistors values in video generation circuit
Signed-off-by: Sergey Kiselev <skiselev@gmail.com>
Parts:
- SW57: value X Ь -> Ь X
- SW66: value CC GRAPH -> CC SHIFT
Changed lines of the file:
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@@
   (title_block
     (title "Radio-86RK")
-    (date "2022-05-11")
-    (rev "1.2")
+    (date "2022-05-13")
+    (rev "1.3")
     (company "Designed by Sergey Kiselev")
     (comment 1 "Based on the previous work by Alexey Khudyakov and Radio magazine publications")
@@
     (in_bom yes) (on_board yes)
     (property "Reference" "SW57" (id 0) (at 128.27 108.966 0))
-    (property "Value" "X Ь" (id 1) (at 124.46 115.57 0))
+    (property "Value" "Ь X" (id 1) (at 124.46 115.57 0))
     (property "Footprint" "Cherry_MX:CHERRY_PCB_100H" (id 2) (at 124.46 111.76 0)
       (effects (font (size 1.27 1.27)) hide)
@@
     (in_bom yes) (on_board yes)
     (property "Reference" "SW66" (id 0) (at 194.31 153.416 0))
-    (property "Value" "CC GRAPH" (id 1) (at 190.5 160.02 0))
+    (property "Value" "CC SHIFT" (id 1) (at 190.5 160.02 0))
     (property "Footprint" "Cherry_MX:CHERRY_PCB_125H" (id 2) (at 190.5 156.21 0)
       (effects (font (size 1.27 1.27)) hide)

Commit message: Add Version 1.4 files
Signed-off-by: Sergey Kiselev <skiselev@gmail.com>
Parts:
- J4: symbol Connector:DIN-8 -> my_components:Conn_DIN-8
- SW10: value ПС LF -> LF ПС
- SW11: value ВК CR -> CR ВК
- SW12: value ЗБ DEL -> DEL ЗБ
- SW2: value СТР CLS -> CLS СТР
- SW3: value АР2 ESC -> ESC АР2
- SW33: value Ю @ -> @ Ю
- SW34: value А A -> A А
- SW35: value Б B -> B Б
- SW36: value Ц C -> C Ц
- SW37: value Д D -> D Д
- SW38: value Е E -> E Е
- SW39: value Ф F -> F Ф
- SW40: value Г G -> G Г
- SW41: value Х H -> H Х
- SW42: value И I -> I И
- SW43: value Й J -> J Й
- SW44: value К K -> K К
- SW45: value Л L -> L Л
- SW46: value М M -> M М
- SW47: value Н N -> N Н
- SW48: value О O -> O О
- SW49: value П P -> P П
- SW50: value Я Q -> Q Я
- SW51: value Р R -> R Р
- SW52: value С S -> S С
- SW53: value Т T -> T Т
- SW54: value У U -> U У
- SW55: value Ж V -> V Ж
- SW56: value В W -> W В
- SW57: value Ь X -> X Ь
- SW58: value Ы Y -> Y Ы
- SW59: value З Z -> Z З
- SW60: value Ш [ -> [ Ш
- SW61: value Э \ -> \ Э
- SW62: value Щ ] -> ] Щ
- SW63: value Ч ^ -> ^ Ч
- SW65: value УС CTRL -> CTRL УС
- SW66: value CC SHIFT -> SHIFT CC
- SW9: value ТАБ TAB -> TAB ТАБ
- U5: symbol my_components:8255 -> my_components:8255A
Connections:
- net GND: now also J4.0
