File: KiCad/Radio-86RK-Power.kicad_sch (KiCad schematic)
At the start: 51 parts, among them J2 5V, J3 Power, U16 7486/К155ЛП5, U17 7474/К155ТМ2, U18 7408/К155ЛИ1, U19 7404/К155ЛН1, U20 7400/К155ЛА3, U25 LM7905/КР1179ЕН5В, U26 IZ0512S

Commit message: Add Version 1.4 files
Signed-off-by: Sergey Kiselev <skiselev@gmail.com>
Parts:
- added J7: Extension, My_Components:Conn_Pin_Header_20x1_2.54mm, symbol Connector_Generic:Conn_01x20
Connections:
- net GND: now also U16.7 (GND), U17.7 (GND), U18.7 (GND), U19.7 (GND), U20.7 (GND), J7.1 (Pin_1), J7.2 (Pin_2)
- net VCC: now also U16.14 (VCC), U17.14 (VCC), U18.14 (VCC), U19.14 (VCC), U20.14 (VCC), J7.10 (Pin_10)
- new net A0: J7.9 (Pin_9)
- new net A1: J7.8 (Pin_8)
- new net A2: J7.7 (Pin_7)
- new net A3: J7.6 (Pin_6)
- new net D0: J7.11 (Pin_11)
- new net D1: J7.12 (Pin_12)
- new net D2: J7.13 (Pin_13)
- new net D3: J7.14 (Pin_14)
- new net D4: J7.15 (Pin_15)
- new net D5: J7.18 (Pin_18)
- new net D6: J7.19 (Pin_19)
- new net D7: J7.20 (Pin_20)
- new net RESET: J7.17 (Pin_17)
- new net TTL_CLK: J7.16 (Pin_16)
- new net ~{EXT_CS}: J7.5 (Pin_5)
- new net ~{RD}: J7.4 (Pin_4)
- new net ~{WR}: J7.3 (Pin_3)
Other:
- note added: "Power Supply and Extension Connector"
- note removed: "Power Supply"
- moved on the sheet: J2, J3
