File: KiCad/Radio-86RK.kicad_sch (KiCad schematic)
At the start: 16 parts, among them SW68 Reset, U1 8080A/КР580ВМ80А, U12 74LS373/К555ИР22, U14 74LS138/К555ИД7, U16 7486/К155ЛП5, U17 7474/К155ТМ2, U18 7408/К155ЛИ1, U19 7404/К155ЛН1, U2 8224/КР580ГФ24, U20 7400/К155ЛА3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

Commit message: Add Version 1.4 files
Signed-off-by: Sergey Kiselev <skiselev@gmail.com>
Parts:
- added LOGO1: Logo_Open_Hardware_Small, Symbol:KiCad-Logo2_6mm_SilkScreen, symbol Graphic:Logo_Open_Hardware_Small
Connections:
- net ~{DMA_CS}: now also U18.1; no longer U18.2
- net at U14.7 (O7): now also U18.2; no longer U18.1
- net ~{EXT_CS}: now reaches U14.10 (O5)
- no-connect marks 11 -> 10
Other:
- sheet Power ports: added ~{EXT_CS}; removed none
- moved on the sheet: U19E
